Commit message: progress

File: ur_app/urdf/ur10e.xacro (robot description, xacro)
@@ -1,8 +1,5 @@
-<?xml version="1.0" ?>
-<!-- =================================================================================== -->
-<!-- |    This document was autogenerated by xacro from /home/afonsocastro/catkin_ws/src/universal_robot/ur_description/urdf/ur10e.xacro | -->
-<!-- |    EDITING THIS FILE BY HAND IS NOT RECOMMENDED                                 | -->
-<!-- =================================================================================== -->
-<robot name="ur10e_robot">
+<?xml version="1.0"?>
+<robot xmlns:xacro="http://wiki.ros.org/xacro">
+    <xacro:macro name="ur10e_robot">
     <!--
     Base UR robot series xacro macro.
@@ -135,10 +132,10 @@
         </inertial>
     </link>
-<!--    Fix the robot to the world-->
-    <link name="world"/>
-    <joint name="fixed" type="fixed">
-        <parent link="world"/>
-        <child link="base_link"/>
-    </joint>
+<!--&lt;!&ndash;    Fix the robot to the world&ndash;&gt;-->
+<!--    <link name="world"/>-->
+<!--    <joint name="fixed" type="fixed">-->
+<!--        <parent link="world"/>-->
+<!--        <child link="base_link"/>-->
+<!--    </joint>-->
     <link name="shoulder_link">
         <visual>
@@ -365,3 +362,4 @@
         </plugin>
     </gazebo>
+    </xacro:macro>
 </robot>
