Commit message: several updates

File: robotiq_2f_140_gripper_visualization/urdf/robotiq_arg2f_140_model_macro.xacro (robot description, xacro)
@@ -1,5 +1,5 @@
 <?xml version="1.0"?>
 <robot xmlns:xacro="http://ros.org/wiki/xacro">
-  <xacro:include filename="$(find robotiq_2f_140_gripper_visualization)/urdf/robotiq_arg2f_transmission.xacro" />
+<!--  <xacro:include filename="$(find robotiq_2f_140_gripper_visualization)/urdf/robotiq_arg2f_transmission.xacro" />-->
   <xacro:macro name="outer_knuckle" params="prefix fingerprefix stroke">
     <link name="${prefix}${fingerprefix}_outer_knuckle">
@@ -154,5 +154,5 @@
   </xacro:macro>
   <xacro:macro name="inner_knuckle_joint" params="prefix fingerprefix reflect">
-    <joint name="${prefix}${fingerprefix}_inner_knuckle_joint" type="revolute">
+    <joint name="${prefix}${fingerprefix}_inner_knuckle_joint" type="fixed">
       <origin xyz="0 ${reflect * -0.0127} 0.06142" rpy="${pi / 2 + .725} 0 ${(reflect - 1) * pi / 2}" />
       <parent link="${prefix}robotiq_arg2f_base_link" />
@@ -164,5 +164,5 @@
   </xacro:macro>
   <xacro:macro name="inner_finger_joint" params="prefix fingerprefix">
-    <joint name="${prefix}${fingerprefix}_inner_finger_joint" type="revolute">
+    <joint name="${prefix}${fingerprefix}_inner_finger_joint" type="fixed">
       <origin xyz="0 0.0817554015893473 -0.0282203446692936" rpy="-0.725 0 0" />
       <parent link="${prefix}${fingerprefix}_outer_finger" />
@@ -183,5 +183,5 @@
   <xacro:include filename="$(find robotiq_2f_140_gripper_visualization)/urdf/robotiq_arg2f.xacro" />
   <xacro:macro name="finger_joint" params="prefix">
-    <joint name="${prefix}finger_joint" type="revolute">
+    <joint name="${prefix}finger_joint" type="fixed">
       <origin xyz="0 -0.030601 0.054905" rpy="${pi / 2 + .725} 0 0" />
       <parent link="${prefix}robotiq_arg2f_base_link" />
@@ -193,5 +193,5 @@
   </xacro:macro>
   <xacro:macro name="right_outer_knuckle_joint" params="prefix">
-    <joint name="${prefix}right_outer_knuckle_joint" type="revolute">
+    <joint name="${prefix}right_outer_knuckle_joint" type="fixed">
       <origin xyz="0 0.030601 0.054905" rpy="${pi / 2 + .725} 0 ${pi}" />
       <parent link="${prefix}robotiq_arg2f_base_link" />
@@ -209,5 +209,5 @@
     <xacro:finger_joint prefix="${prefix}"/>
     <xacro:right_outer_knuckle_joint prefix="${prefix}"/>
-    <xacro:robotiq_arg2f_transmission prefix="${prefix}"/>
+<!--    <xacro:robotiq_arg2f_transmission prefix="${prefix}"/>-->
   </xacro:macro>
 </robot>

File: robotiq_2f_140_gripper_visualization/urdf/robotiq_arg2f_transmission.xacro (robot description, xacro)
@@ -1,14 +1,14 @@
-<?xml version="1.0"?>
-<robot xmlns:xacro="http://ros.org/wiki/xacro">
-  <xacro:macro name="robotiq_arg2f_transmission" params="prefix">
-    <transmission name="${prefix}finger_joint_trans">
-      <type>transmission_interface/SimpleTransmission</type>
-      <joint name="${prefix}finger_joint">
-        <hardwareInterface>PositionJointInterface</hardwareInterface>
-      </joint>
-      <actuator name="${prefix}finger_joint_motor">
-        <mechanicalReduction>1</mechanicalReduction>
-      </actuator>
-    </transmission>
-  </xacro:macro>
-</robot>
+<!--<?xml version="1.0"?>-->
+<!--<robot xmlns:xacro="http://ros.org/wiki/xacro">-->
+<!--  <xacro:macro name="robotiq_arg2f_transmission" params="prefix">-->
+<!--    <transmission name="${prefix}finger_joint_trans">-->
+<!--      <type>transmission_interface/SimpleTransmission</type>-->
+<!--      <joint name="${prefix}finger_joint">-->
+<!--        <hardwareInterface>PositionJointInterface</hardwareInterface>-->
+<!--      </joint>-->
+<!--      <actuator name="${prefix}finger_joint_motor">-->
+<!--        <mechanicalReduction>1</mechanicalReduction>-->
+<!--      </actuator>-->
+<!--    </transmission>-->
+<!--  </xacro:macro>-->
+<!--</robot>-->

File: scripts/urdf/ur10e.xacro (robot description, xacro)
@@ -1,5 +1,8 @@
-<?xml version="1.0"?>
-<robot xmlns:xacro="http://wiki.ros.org/xacro">
-    <xacro:macro name="ur10e_robot">
+<?xml version="1.0" ?>
+<!-- =================================================================================== -->
+<!-- |    This document was autogenerated by xacro from /home/afonsocastro/catkin_ws/src/MecInTouch_workshop/ur_description/urdf/ur10e.xacro | -->
+<!-- |    EDITING THIS FILE BY HAND IS NOT RECOMMENDED                                 | -->
+<!-- =================================================================================== -->
+<robot xmlns:xacro="http://wiki.ros.org/xacro" name="ur10e_robot">
     <!--
     Base UR robot series xacro macro.
@@ -48,4 +51,23 @@
           this location. Nor can they rely on the existence of the macro.
   -->
+    <xacro:property name="M_PI" value="3.1415926535897931"/>
+            <!-- Tables properties-->
+    <xacro:property name="table_height" value="0.795"/>
+    <xacro:property name="table_width" value=".9"/>
+    <xacro:property name="table_length" value="1.25"/>
+    <xacro:property name="table_tabletop_thickness" value="0.015"/>
+    <xacro:property name="table_leg_radius" value="0.02"/>
+    <!-- Gantry properties-->
+    <xacro:property name="gantry_height" value="2.29"/>
+    <xacro:property name="gantry_foot_height" value="0.065"/>
+    <xacro:property name="gantry_width" value="4"/>
+    <xacro:property name="gantry_length" value="2.7975"/>
+    <xacro:property name="gantry_thickness" value="0"/>
+    <xacro:property name="gantry_leg_radius" value="0.09"/>
+    <xacro:include filename="$(find ur_description)/urdf/table.macro.xacro"/>
+    <xacro:include filename="$(find ur_description)/urdf/gantry.macro.xacro"/>
+    <xacro:include filename="$(find ur_description)/urdf/astra.urdf.xacro"/>
+    <xacro:include filename="$(find robotiq_2f_140_gripper_visualization)/urdf/robotiq_arg2f_140_model.xacro" />
+    <xacro:include filename="$(find ur_description)/urdf/wood_block.macro.xacro"/>
     <transmission name="shoulder_pan_trans">
         <type>transmission_interface/SimpleTransmission</type>
@@ -132,6 +154,28 @@
         </inertial>
     </link>
-<!--&lt;!&ndash;    Fix the robot to the world&ndash;&gt;-->
-<!--    <link name="world"/>-->
+    <link name="world"/>
+    <joint name="world_to_robot_joint" type="fixed">
+        <parent link="tabletop_table_base"/>
+        <child link="base_link"/>
+        <origin xyz="0 0 -0.015" rpy="0 0 0"/>
+    </joint>
+    <xacro:table_macro name="table_base" parent="world" width="${table_width}"
+                       length="${table_length}" height="${table_height}"
+                       tabletop_thickness="${table_tabletop_thickness}" leg_radius="${table_leg_radius}">
+        <origin xyz="0.1 ${gantry_length/2-table_width/2} 0" rpy="0 0 ${-M_PI/2}"/>
+    </xacro:table_macro>
+    <xacro:gantry_macro name="gantry" parent="world" width="${gantry_width}"
+                        length="${gantry_length}" height="${gantry_height}" foot_height="${gantry_foot_height}"
+                        gantry_thickness="${gantry_thickness}" leg_radius="${gantry_leg_radius}">
+        <origin xyz="0 0 0" rpy="0 0 0"/>
+    </xacro:gantry_macro>
+    <xacro:sensor_astra prefix="camera_top" parent="world">
+        <origin xyz="0.09511408182797733 0.14905972847160784 2.4330682231422602"
+                rpy="-1.9962039976135075 1.491251777066553 -2.0400319820116386"/>
+    </xacro:sensor_astra>
+    <xacro:sensor_astra prefix="camera_right" parent="world">
+        <origin xyz="-0.47389933117248495 0.6050706033175103 1.2510900165155419"
+                rpy="0.1688160669718149 0.3885697035429511 -0.6796268633018927"/>
+    </xacro:sensor_astra>
 <!--    <joint name="fixed" type="fixed">-->
 <!--        <parent link="world"/>-->
@@ -362,4 +406,89 @@
         </plugin>
     </gazebo>
-    </xacro:macro>
+    <xacro:wood_block_macro parent="world">
+        <origin xyz="0 0 0.835" rpy="0 0 ${M_PI}"/>
+    </xacro:wood_block_macro>
+    <joint name="tool0-FT_sensor_base" type="fixed">
+        <parent link="tool0"/>
+        <child link="FT_sensor_base"/>
+        <origin xyz="0 0 0.007" rpy="0 0 ${M_PI/2}"/>
+    </joint>
+    <link name="FT_sensor_base">
+        <visual>
+          <geometry>
+            <cylinder length="0.014" radius="0.05"/>
+          </geometry>
+          <material name="metalic_blue">
+            <color rgba="0.0118 0.5176 0.6706 1.0"/>
+          </material>
+        </visual>
+        <collision>
+          <geometry>
+            <cylinder length="0.014" radius="0.05"/>
+          </geometry>
+        </collision>
+    </link>
+    <joint name="FT_sensor_base-FT_sensor" type="fixed">
+        <parent link="FT_sensor_base"/>
+        <child link="FT_sensor"/>
+        <origin xyz="0 0 0.0215" rpy="0 0 0"/>
+    </joint>
+    <link name="FT_sensor">
+        <visual>
+          <geometry>
+            <cylinder length="0.029" radius="0.04"/>
+          </geometry>
+          <material name="metalic_blue">
+            <color rgba="0.0118 0.5176 0.6706 1.0"/>
+          </material>
+          <gazebo>
+            <material>Gazebo/Blue</material>
+          </gazebo>
+        </visual>
+        <collision>
+          <geometry>
+            <cylinder length="0.029" radius="0.04"/>
+          </geometry>
+        </collision>
+    </link>
+    <joint name="gripper_joint" type="fixed">
+        <parent link="FT_sensor"/>
+        <child link="robotiq_arg2f_base_link"/>
+        <origin xyz="0 0 0.0215" rpy="0 0 0"/>
+    </joint>
+    <xacro:table_macro name="table_front" parent="table_base" width="0.7"
+                       length="1.20" height="0.75"
+                       tabletop_thickness="0.015" leg_radius="0.02">
+        <origin xyz="${(0.9+0.7)/2} 0 0" rpy="0 0 0"/>
+    </xacro:table_macro>
+<!--    <link name="table_beam">-->
+<!--        <visual>-->
+<!--            <origin xyz="0.0 0.0 0.0" rpy="0 0 0" />-->
+<!--            <geometry>-->
+<!--                <mesh filename="package://ur_description/meshes/bosch_40x40x150.STL" scale="0.001 0.01 0.001" />-->
+<!--            </geometry>-->
+<!--            <material name="grey">-->
+<!--                <color rgba="0.678 0.678 0.678 1.0"/>-->
+<!--            </material>-->
+<!--&lt;!&ndash;            <material name="grey"/>&ndash;&gt;-->
+<!--        </visual>-->
+<!--        <collision>-->
+<!--            <origin xyz="0.02 0.75 0.02" rpy="${M_PI/2} 0 0" />-->
+<!--            <geometry>-->
+<!--                <box size="0.05 0.05 1.55"/>-->
+<!--            </geometry>-->
+<!--        </collision>-->
+<!--        <inertial>-->
+<!--            <mass value="1.0" />-->
+<!--            <origin xyz="0.0 0.0 ${0.75/2-40-0.001}" rpy="0 0 0" />-->
+<!--            <inertia ixx="0.1" ixy="0"  ixz="0"-->
+<!--                     iyy="0.1" iyz="0"-->
+<!--                     izz="0.01" />-->
+<!--        </inertial>-->
+<!--    </link>-->
+<!--    <joint name="table_base_to_table_beam" type="fixed">-->
+<!--        <parent link="table_base" />-->
+<!--        <child link="table_beam" />-->
+<!--        <origin xyz="0.308 -0.625 0.0035" rpy="${M_PI/2} 0 0"/>-->
+<!--    </joint>-->
 </robot>
